File: PCB files/UnderglowPCB/UnderglowPCB.sch (KiCad schematic (older format))
At the start: 37 parts, among them J1 Screw_Terminal_01x03, J10 Conn_01x07, J2 Screw_Terminal_01x03, J3 Screw_Terminal_01x03, J4 Screw_Terminal_01x03, J5 Screw_Terminal_01x03, J6 Screw_Terminal_01x03, J7 Screw_Terminal_01x03, J8 Conn_01x05, J9 Screw_Terminal_01x02, SW1 SW_Push, U1 74HC14, U2 74HC14, U3 74HC14, U4 74HC14, U5 74HC14, U6 74HC14

Commit message: PCB rev 1 schematic complete, custom footprint done.
Parts:
- removed C2: 2.2UF-X7R_0805, symbol OPL_Capacitor:CERAMIC-2.2UF-25V-10%-X7R_0805_
- removed C5: 2.2uF-x7r_0805, symbol OPL_Capacitor:CERAMIC-2.2UF-25V-10%-X7R_0805_
- removed J9: Screw_Terminal_01x02, symbol Connector:Screw_Terminal_01x02
- removed R5: 27k, symbol Device:R
- removed R6: 10k, symbol Device:R
- removed U3: 74HC14, symbol Regulator_Switching:TPS62133
- removed U4: 74HC14, symbol RF_Module:ESP32-WROOM-32D
- added C1, C2, C3, C4, C7, C9: 10u, symbol Device:C_Small
- added C11, C13: 2.2u, symbol Device:C_Small
- added D1, D2: LED, symbol Device:LED
- added D3: BAT760-7, symbol Device:D_Schottky
- added D4: RB088BM-60TL, symbol Device:D_Schottky
- added F1: Fuse, symbol Device:Fuse
- added FB1: Ferrite_Bead_Small, symbol Device:Ferrite_Bead_Small
- added H1, H2, H3, H4: MH_Pad, symbol Mechanical:MountingHole_Pad
- added J1: USB_B_Micro, symbol Connector:USB_B_Micro
- added J11: Screw_Terminal_01x02, symbol Connector:Screw_Terminal_01x02
- added J12: DB9_Male, symbol Connector:DB9_Male
- added Q1, Q2: S8050, Package_TO_SOT_THT:TO-92_Inline, symbol Transistor_BJT:S8050
- added R1, R2: 2.2k, symbol Device:R
- added R10, R12, R13, R9: 10k, symbol Device:R
- added R7: 4.7k, symbol Device:R
- added R8: 27k, symbol Device:R
- added U1: CP2102N-A01-GQFN28, Package_DFN_QFN:QFN-28-1EP_5x5mm_P0.5mm_EP3.35x3.35mm, symbol Interface_USB:CP2102N-A01-GQFN28
- added U2: TPS62133, Package_DFN_QFN:VQFN-16-1EP_3x3mm_P0.5mm_EP1.68x1.68mm_ThermalVias, symbol Regulator_Switching:TPS62133
- added U6: ESP32-WROOM-32D, RF_Module:ESP32-WROOM-32, symbol RF_Module:ESP32-WROOM-32D
- C10: renamed from C6; symbol pspice:C -> Device:C_Small
- C12, C14, C15, C16, C17: renamed from C?; symbol pspice:C -> Device:C_Small
- C5: renamed from C1; symbol pspice:C -> Device:C_Small
- C6: renamed from C3; symbol pspice:C -> Device:C_Small
- C8: renamed from C4; symbol pspice:C -> Device:C_Small
- J6: renamed from J7; value Screw_Terminal_01x03 -> Screw_Terminal_01x04; symbol Connector:Screw_Terminal_01x03 -> Connector:Screw_Terminal_01x04
- U5: renamed from U1; value 74HC14 -> LD56100DPU33R
- U7: renamed from U2; value 74HC14 -> SN65HVD230
- renumbered J6 to J10, J1 to J2, J2 to J3, J10 to J4, J8 to J5, J3 to J7, J4 to J8, J5 to J9, R2 to R11, R1 to R14, R7 to R5, R8 to R6, U5 to U3, U6 to U4
Connections:
- net labels added: +12V, BRAKE_LOW, EN, IO0, PROG_DTR, PROG_RTS, RXD0, TURN_LEFT_LOW, TURN_RIGHT_LOW, TXD0, UG_LOW_FRONT, UG_LOW_LEFT, UG_LOW_REAR, UG_LOW_RIGHT, UG_LOW_SPARE_1, UG_LOW_SPARE_2
- net labels removed: +12V_BATT, MISO
- wire segments 166 -> 177
- no-connect marks 9 -> 32
Other:
- note added: "Board Power (12v)"
- note added: "KiCAD complains about pins 1 & 2.\nPins are correct: IC Outputs to both pins"
- note added: "Mounting Holes"
- note added: "PWR LEDs"
- note added: "Programming switch mode"
- note added: "Schmitt 3.3v to 5v logic"
- note added: "Shmitt 3.3v to 5v power"
- note added: "Turn Signal & Brake\n12v to 3.3v"
- note added: "USB to UART\nConnector"
- note added: "Using ESP-32 WROOM 32E\nE is drop in replacement for D"
- note removed: "Controller"
- note removed: "Note: Some GPIO identities (GPIO 39, etc) are relabeled."
- moved on the sheet: J10, J2, J3, J4, J5, J7, J8, J9, L1, R11, R14, R3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
